File: Way to silence/I2SAmp.kicad_sch (KiCad schematic)
At the start: 8 parts, among them U4 MAX98357AETE+T

Commit message: [ADD] Screw Connector
Parts:
- added J2: Screw_Terminal_01x02, symbol Way to silence:Screw_Terminal_01x02
Connections:
- net at C5.2, FB2.2: now also J2.2 (Pin_2)
- net at C6.2, FB1.2: now also J2.1 (Pin_1)
Other:
- note added: "+"
- note added: "-"
Changed lines of the file:
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@@
     (stroke (width 0) (type default))
+  )
+  (text "-" (at 142.24 57.15 0)
+    (effects (font (size 1.27 1.27)) (justify left bottom))
+  )
+  (text "+\n" (at 142.24 59.69 0)
+    (effects (font (size 1.27 1.27)) (justify left bottom))
   )
   (hierarchical_label "DIN" (shape bidirectional) (at 22.86 20.32 180) (fields_autoplaced)
@@
         )
       )
+    )
+  )
+  (symbol (lib_id "Way to silence:Screw_Terminal_01x02") (at 139.7 55.88 0) (unit 1)
+    (in_bom yes) (on_board yes) (dnp no)
+    (property "Reference" "J2" (at 138.43 49.53 0)
+      (effects (font (size 1.27 1.27)) (justify left))
+    )
+    (property "Value" "Screw_Terminal_01x02" (at 129.54 52.07 0)
+      (effects (font (size 1.27 1.27)) (justify left))
+    )
+    (property "Footprint" "" (at 139.7 55.88 0)
+      (effects (font (size 1.27 1.27)) hide)
+    )
+    (property "Datasheet" "~" (at 139.7 55.88 0)
+      (effects (font (size 1.27 1.27)) hide)
+    )
+    (pin "1")
+    (pin "2")
+    (instances
+      (project "Way to silence"
+        (path "/9822a1be-a034-44c3-8530-56368958b215/7708567a-63f7-491b-967e-673f1a10dffd"
+          (reference "J2") (unit 1)
+        )
+      )

Commit message: [DRC] I2S Amp seems Sheet ok
Parts:
- renumbered C5 to C?, C6 to C?, FB2 to FB?, FB1 to FB?, U4 to U?
Connections:
- net GND: now also U?.17 (EP)
- no-connect marks 0 -> 4
Other:
- moved on the sheet: C7, C8, C?, FB?, J2, R11, U?

Commit message: [ADD] LSCS Parts and Footprints for BMS
Parts:
- C7, C8, C? (x2): footprint (none) -> Way to silence:C_0603_1608Metric
- R11: footprint (none) -> Way to silence:R_0603_1608Metric
Changed lines of the file:
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@@
       (effects (font (size 1.27 1.27)) (justify right))
     )
-    (property "Footprint" "" (at 115.8748 49.53 90)
+    (property "Footprint" "Way to silence:C_0603_1608Metric" (at 115.8748 49.53 90)
       (effects (font (size 1.27 1.27)) hide)
     )
@@
       (effects (font (size 1.27 1.27)))
     )
-    (property "Footprint" "" (at 39.37 38.608 0)
+    (property "Footprint" "Way to silence:R_0603_1608Metric" (at 39.37 38.608 0)
       (effects (font (size 1.27 1.27)) hide)
     )
@@
       (effects (font (size 1.27 1.27)) (justify right))
     )
-    (property "Footprint" "" (at 33.3248 46.99 90)
+    (property "Footprint" "Way to silence:C_0603_1608Metric" (at 33.3248 46.99 90)
       (effects (font (size 1.27 1.27)) hide)
     )
@@
       (effects (font (size 1.27 1.27)) (justify right))
     )
-    (property "Footprint" "" (at 128.5748 49.53 90)
+    (property "Footprint" "Way to silence:C_0603_1608Metric" (at 128.5748 49.53 90)
       (effects (font (size 1.27 1.27)) hide)
     )
@@
       (effects (font (size 1.27 1.27)) (justify right))
     )
-    (property "Footprint" "" (at 44.7548 46.99 90)
-      (effects (font (size 1.27 1.27)) hide)
-    )
+    (property "Footprint" "Way to silence:C_0603_1608Metric" (at 44.7548 46.99 90)
+      (effects (font (size 1.27 1.27)) hide)
+    )

Commit message: [ADD] References in readme
Parts:
- J2: footprint (none) -> Way to silence:Screw_Terminal_3.5; LCSC (none) -> C784942
Changed lines of the file:
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@@
       (effects (font (size 1.27 1.27)) (justify left))
     )
-    (property "Footprint" "" (at 139.7 44.45 0)
+    (property "Footprint" "Way to silence:Screw_Terminal_3.5" (at 139.7 35.56 0)
       (effects (font (size 1.27 1.27)) hide)
     )
@@
       (effects (font (size 1.27 1.27)) hide)
     )
+    (property "LCSC" "C784942" (at 139.7 33.02 0)
+      (effects (font (size 1.27 1.27)) hide)
+    )

Commit message: [UPDT] Switch source
Parts:
- C7: LCSC (none) -> C14663
- C8: LCSC (none) -> C77041
Changed lines of the file:
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@@
+      (effects (font (size 1.27 1.27)) hide)
+    )
+    (property "LCSC" "C77041" (at 34.29 50.8 90)
       (effects (font (size 1.27 1.27)) hide)
     )
@@
       (effects (font (size 1.27 1.27)) hide)
     )
+    (property "LCSC" "C14663" (at 45.72 50.8 90)
+      (effects (font (size 1.27 1.27)) hide)
+    )

Commit message: [ADD] I2S Amp LSCS Refs
Parts:
- C? (x2): LCSC (none) -> C1603
- FB? (x2): LSCS (none) -> C394474
- R11: LSCS (none) -> C22935
Changed lines of the file:
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@@
+      (effects (font (size 1.27 1.27)) hide)
+    )
+    (property "LCSC" "C1603" (at 116.84 53.34 90)
       (effects (font (size 1.27 1.27)) hide)
     )
@@
       (effects (font (size 1.27 1.27)) hide)
     )
+    (property "LSCS" "C22935" (at 39.37 36.83 0)
+      (effects (font (size 1.27 1.27)) hide)
+    )
     (pin "1")
     (pin "2")
@@
     )
     (property "Datasheet" "~" (at 106.68 44.45 90)
+      (effects (font (size 1.27 1.27)) hide)
+    )
+    (property "LSCS" "C394474" (at 106.68 44.45 0)
       (effects (font (size 1.27 1.27)) hide)
     )
@@
       (effects (font (size 1.27 1.27)) hide)
     )
+    (property "LSCS" "C394474" (at 106.68 57.15 0)
+      (effects (font (size 1.27 1.27)) hide)
+    )
     (pin "1")
     (pin "2")
@@
       (effects (font (size 1.27 1.27)) hide)
     )
+    (property "LCSC" "C1603" (at 129.54 53.34 90)
+      (effects (font (size 1.27 1.27)) hide)
+    )

Commit message: [ADD] Missing footprints
Parts:
- FB? (x2): footprint (none) -> Way to silence:Inductor; LCSC (none) -> C2847468; LSCS C394474 -> (none)
Changed lines of the file:
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@@
       (effects (font (size 1.27 1.27)))
     )
-    (property "Footprint" "" (at 106.68 46.228 0)
+    (property "Footprint" "Way to silence:Inductor" (at 106.68 46.228 0)
       (effects (font (size 1.27 1.27)) hide)
     )
@@
       (effects (font (size 1.27 1.27)) hide)
     )
-    (property "LSCS" "C394474" (at 106.68 44.45 0)
+    (property "LCSC" "C2847468" (at 106.68 44.45 0)
       (effects (font (size 1.27 1.27)) hide)
     )
@@
     )
   )
-  (symbol (lib_id "Way to silence:FerriteBead") (at 106.68 57.15 0) (unit 1)
+  (symbol (lib_name "FerriteBead_1") (lib_id "Way to silence:FerriteBead") (at 106.68 57.15 0) (unit 1)
     (in_bom yes) (on_board yes) (dnp no)
     (property "Reference" "FB?" (at 106.6292 49.53 0)
@@
       (effects (font (size 1.27 1.27)))
     )
-    (property "Footprint" "" (at 106.68 58.928 0)
+    (property "Footprint" "Way to silence:Inductor" (at 106.68 58.928 0)
       (effects (font (size 1.27 1.27)) hide)
     )
@@
       (effects (font (size 1.27 1.27)) hide)
     )
-    (property "LSCS" "C394474" (at 106.68 57.15 0)
+    (property "LCSC" "C2847468" (at 106.68 48.26 0)
       (effects (font (size 1.27 1.27)) hide)
     )

Commit message: [ADD] Beg of routing
Parts:
- J2: value Screw_Terminal_01x02 -> Amplificator_Terminal
Changed lines of the file:
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@@
       (effects (font (size 1.27 1.27)) (justify left))
     )
-    (property "Value" "Screw_Terminal_01x02" (at 129.54 40.64 0)
+    (property "Value" "Amplificator_Terminal" (at 129.54 40.64 0)
       (effects (font (size 1.27 1.27)) (justify left))
     )
