File: Way to silence/_autosave-Way to silence.kicad_sch (KiCad schematic)
At the start: 17 parts, among them J3 5V_Terminal, J4 Battery_Terminal, J5 LEDS Port, SW1 SW_SPDT, SW3 SW_SPST, U1 ESP32-WROOM-32-N16, U6 AMS1117CD-3.3

Commit message: [ADD] Pin header for leds
Parts:
- J5: footprint (none) -> Way to silence:PinHeader_1x03_P2.54mm_Vertical
Changed lines of the file:
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@@
       (effects (font (size 1.27 1.27)))
     )
-    (property "Footprint" "" (at 82.55 93.98 0)
+    (property "Footprint" "Way to silence:PinHeader_1x03_P2.54mm_Vertical" (at 82.55 93.98 0)
       (effects (font (size 1.27 1.27)) hide)
     )
