File: Way to silence/USB to Uart.kicad_sch (KiCad schematic)
At the start: 12 parts, among them Q1 BC817, Q2 BC817, U5 USB-TYPE-C-018

Commit message: [UDPT] Schematics from testings
Parts:
- added C21: 10uF, Way to silence:C_0603_1608Metric, symbol Way to silence:C
- added R21: 10K, Way to silence:R_0603_1608Metric, symbol Way to silence:R
Connections:
- net +3.3V: now also R21.1
- net EN: now also C21.2, R21.2
- net GND: now also C21.1
- net RXD: now also U?.26 (TXD); no longer U?.25 (RXD)
- net TXD: now also U?.25 (RXD); no longer U?.26 (TXD)
Other:
- note removed: "+"
- note removed: "-"
- note removed: "10KR"
- note removed: "10uF"
